Commit message: 完善amcl与liosam配合实现自动定位

File: LIO-SAM_MID360_ROS2_PKG/ros2/install/lio_sam/share/lio_sam/config/robot.urdf.xacro (robot description, xacro)
@@ -1,35 +1 @@
-<?xml version="1.0"?>
-<robot name="lio" xmlns:xacro="http://tixiaoshan.github.io/">
-  <xacro:property name="PI" value="3.1415926535897931" />
-  <link name="chassis_link"></link>
-  <link name="base_link"></link>
-  <joint name="base_link_joint" type="fixed">
-    <parent link="base_link"/>
-    <child link="chassis_link" />
-    <origin xyz="0 0 0" rpy="0 0 0" />
-  </joint>
-  <link name="livox_frame"> </link>
-  <joint name="lidar_joint" type="fixed">
-    <parent link="base_link" />
-    <child link="livox_frame" />
-    <origin xyz="0 0 0" rpy="0 0 0" />
-  </joint>
-  <link name="imu_link"> </link>
-  <joint name="imu_joint" type="fixed">
-    <parent link="chassis_link" />
-    <child link="imu_link" />
-    <origin xyz="0 0 0" rpy="0 0 0" />
-  </joint>
-  <link name="laser_sensor_frame"> </link>
-  <joint name="laser_joint" type="fixed">
-    <parent link="imu_link" />
-    <child link="laser_sensor_frame" />
-    <origin xyz="0 0 0" rpy="0 0 0" />
-  </joint>
-  <link name="navsat_link"> </link>
-  <joint name="navsat_joint" type="fixed">
-    <parent link="chassis_link" />
-    <child link="navsat_link" />
-    <origin xyz="0 0 0" rpy="0 0 0" />
-  </joint>
-</robot>
+/home/ywj/projects/git/dog_slam/LIO-SAM_MID360_ROS2_PKG/ros2/src/LIO-SAM_MID360_ROS2_DOG/config/robot.urdf.xacro
