Commit message: change to online mode

File: LIO-SAM_MID360_ROS2_PKG/ros2/src/LIO-SAM_MID360_ROS2_DOG/config/robot.urdf.xacro (robot description, xacro)
@@ -13,5 +13,5 @@
     <parent link="base_link" />
     <child link="livox_frame" />
-    <origin xyz="0 0 0" rpy="0 0 0" />
+    <origin xyz="0 0 0" rpy="0 ${PI/6} 0" /> <!-- 激光雷达前倾30度 -->
   </joint>
   <link name="imu_link"> </link>

Commit message: 针对不同电脑使用不同配置，恢复雷达角度

File: LIO-SAM_MID360_ROS2_PKG/ros2/src/LIO-SAM_MID360_ROS2_DOG/config/robot.urdf.xacro (robot description, xacro)
@@ -13,5 +13,6 @@
     <parent link="base_link" />
     <child link="livox_frame" />
-    <origin xyz="0 0 0" rpy="0 ${PI/6} 0" /> <!-- 激光雷达前倾30度 -->
+    <!-- <origin xyz="0 0 0" rpy="0 ${PI/6} 0" /> 激光雷达前倾30度 -->
+    <origin xyz="0 0 0" rpy="0 0 0" />
   </joint>
   <link name="imu_link"> </link>

Commit message: 改进bt navigator参数

File: LIO-SAM_MID360_ROS2_PKG/ros2/src/LIO-SAM_MID360_ROS2_DOG/config/robot.urdf.xacro (robot description, xacro)
@@ -13,24 +13,12 @@
     <parent link="base_link" />
     <child link="livox_frame" />
-    <!-- <origin xyz="0 0 0" rpy="0 ${PI/6} 0" /> 激光雷达前倾30度 -->
-    <origin xyz="0 0 0" rpy="0 0 0" />
+    <origin xyz="0 0 0" rpy="0 ${PI/6} 0" /> 激光雷达前倾30度
+    <!-- <origin xyz="0 0 0" rpy="0 0 0" /> -->
   </joint>
   <link name="imu_link"> </link>
   <joint name="imu_joint" type="fixed">
-    <parent link="chassis_link" />
+    <parent link="base_link" />
     <child link="imu_link" />
-    <origin xyz="0 0 0" rpy="0 0 0" />
-  </joint>
-  <link name="laser_sensor_frame"> </link>
-  <joint name="laser_joint" type="fixed">
-    <parent link="imu_link" />
-    <child link="laser_sensor_frame" />
-    <origin xyz="0 0 0" rpy="0 0 0" />
-  </joint>
-  <link name="navsat_link"> </link>
-  <joint name="navsat_joint" type="fixed">
-    <parent link="chassis_link" />
-    <child link="navsat_link" />
-    <origin xyz="0 0 0" rpy="0 0 0" />
+    <origin xyz="0 0 0" rpy="0 ${PI/6} 0" />
   </joint>
 </robot>

Commit message: 优化

File: LIO-SAM_MID360_ROS2_PKG/ros2/src/LIO-SAM_MID360_ROS2_DOG/config/robot.urdf.xacro (robot description, xacro)
@@ -13,6 +13,6 @@
     <parent link="base_link" />
     <child link="livox_frame" />
-    <origin xyz="0 0 0" rpy="0 ${PI/6} 0" /> 激光雷达前倾30度
-    <!-- <origin xyz="0 0 0" rpy="0 0 0" /> -->
+    <!-- <origin xyz="0 0 0" rpy="0 ${PI/6} 0" /> 激光雷达前倾30度 -->
+    <origin xyz="0 0 0" rpy="0 0 0" />
   </joint>
   <link name="imu_link"> </link>
@@ -20,5 +20,6 @@
     <parent link="base_link" />
     <child link="imu_link" />
-    <origin xyz="0 0 0" rpy="0 ${PI/6} 0" />
+    <origin xyz="0 0 0" rpy="0 0 0" />
+    <!-- <origin xyz="0 0 0" rpy="0 ${PI/6} 0" /> -->
   </joint>
 </robot>
