Commit message: 根据现场情况优化参数，特别是雷达距离和姿态限制

File: LIO-SAM_MID360_ROS2_PKG/ros2/src/LIO-SAM_MID360_ROS2_DOG/config/robot.urdf_tilt.xacro (robot description, xacro)
@@ -3,23 +3,16 @@
   <xacro:property name="PI" value="3.1415926535897931" />
   <link name="chassis_link"></link>
-  <link name="base_link"></link>
+  <!-- <link name="base_link"></link>
   <joint name="base_link_joint" type="fixed">
     <parent link="base_link"/>
     <child link="chassis_link" />
     <origin xyz="0 0 0" rpy="0 0 0" />
-  </joint>
+  </joint> -->
   <link name="livox_frame"> </link>
   <joint name="lidar_joint" type="fixed">
     <parent link="base_link" />
     <child link="livox_frame" />
-    <origin xyz="0 0 0" rpy="0 ${PI/6} 0" /> 激光雷达前倾30度
+    <origin xyz="0 0 0" rpy="0 ${PI/6} 0" />
     <!-- <origin xyz="0 0 0" rpy="0 0 0" /> -->
   </joint>
-  <link name="imu_link"> </link>
-  <joint name="imu_joint" type="fixed">
-    <parent link="base_link" />
-    <child link="imu_link" />
-    <!-- <origin xyz="0 0 0" rpy="0 0 0" /> -->
-    <origin xyz="0 0 0" rpy="0 ${PI/6} 0" />
-  </joint>
 </robot>

Commit message: sync

File: LIO-SAM_MID360_ROS2_PKG/ros2/src/LIO-SAM_MID360_ROS2_DOG/config/robot.urdf_tilt.xacro (robot description, xacro)
@@ -2,11 +2,5 @@
 <robot name="lio" xmlns:xacro="http://tixiaoshan.github.io/">
   <xacro:property name="PI" value="3.1415926535897931" />
-  <link name="chassis_link"></link>
-  <!-- <link name="base_link"></link>
-  <joint name="base_link_joint" type="fixed">
-    <parent link="base_link"/>
-    <child link="chassis_link" />
-    <origin xyz="0 0 0" rpy="0 0 0" />
-  </joint> -->
+  <link name="base_link"></link>
   <link name="livox_frame"> </link>
   <joint name="lidar_joint" type="fixed">
@@ -16,3 +10,10 @@
     <!-- <origin xyz="0 0 0" rpy="0 0 0" /> -->
   </joint>
+  <link name="lidar_link"> </link>
+  <joint name="lidar_link_joint" type="fixed">
+    <parent link="base_link" />
+    <child link="lidar_link" />
+    <origin xyz="0 0 0" rpy="0 0 0" />
+    <!-- <origin xyz="0 0 0" rpy="0 0 0" /> -->
+  </joint>
 </robot>

Commit message: 调整激光雷达tf角度，存在看不到laserscan的问题，但是数值正确

File: LIO-SAM_MID360_ROS2_PKG/ros2/src/LIO-SAM_MID360_ROS2_DOG/config/robot.urdf_tilt.xacro (robot description, xacro)
@@ -14,5 +14,5 @@
     <parent link="base_link" />
     <child link="lidar_link" />
-    <origin xyz="0 0 0" rpy="0 0 0" />
+    <origin xyz="0 0 0" rpy="0 ${PI/6} 0" />
     <!-- <origin xyz="0 0 0" rpy="0 0 0" /> -->
   </joint>

Commit message: 导航已稳定，但是可能定位会突然飘

File: LIO-SAM_MID360_ROS2_PKG/ros2/src/LIO-SAM_MID360_ROS2_DOG/config/robot.urdf_tilt.xacro (robot description, xacro)
@@ -7,5 +7,5 @@
     <parent link="base_link" />
     <child link="livox_frame" />
-    <origin xyz="0 0 0" rpy="0 ${PI/6} 0" />
+    <origin xyz="0.1 0 0.1" rpy="0 ${PI/6} 0" />
     <!-- <origin xyz="0 0 0" rpy="0 0 0" /> -->
   </joint>
@@ -14,5 +14,5 @@
     <parent link="base_link" />
     <child link="lidar_link" />
-    <origin xyz="0 0 0" rpy="0 ${PI/6} 0" />
+    <origin xyz="0.1 0 0.1" rpy="0 ${PI/6} 0" />
     <!-- <origin xyz="0 0 0" rpy="0 0 0" /> -->
   </joint>
