Commit message: 修正模型加载问题

File: LIO-SAM_MID360_ROS2_PKG/ros2/src/ros2_livox_simulation/urdf/my_robot/sensor/mid360.xacro (robot description, xacro)
@@ -24,5 +24,5 @@
         <origin xyz="0.025 -0.0265 -0.025" rpy="${pi/2} 0 ${pi}"/>
         <geometry>
-          <mesh filename="/home/ywj/dog_slam/LIO-SAM_MID360_ROS2_PKG/ros2/src/ros2_livox_simulation/meshes/mid360.stl" scale="0.0008 0.0008 0.0008"/>
+          <mesh filename="package://ros2_livox_simulation/meshes/mid360.stl" scale="0.0008 0.0008 0.0008"/>
         </geometry>
       </visual>
@@ -30,5 +30,5 @@
     <origin xyz="0.025 -0.0265 -0.025" rpy="${pi/2} 0 ${pi}"/>
     <geometry>
-      <mesh filename="/home/ywj/dog_slam/LIO-SAM_MID360_ROS2_PKG/ros2/src/ros2_livox_simulation/meshes/mid360.stl" scale="0.0008 0.0008 0.0008"/>
+      <mesh filename="package://ros2_livox_simulation/meshes/mid360.stl" scale="0.0008 0.0008 0.0008"/>
     </geometry>
   </collision>
