Commit message: gazebo with fastlio2+nav2

File: LIO-SAM_MID360_ROS2_PKG/ros2/src/ros2_livox_simulation/urdf/my_robot/my_robot.xacro (robot description, xacro)
@@ -63,5 +63,5 @@
 <!-- =============== 轮子配置 =============== -->
 <!-- =============== mid360 ============ -->
-  <xacro:mid360  name="livox_frame" parent="base_link" topic="/livox">
+  <xacro:mid360  name="livox_frame" parent="base_link" topic="/livox/lidar">
     <origin xyz="0.0 0.0 0.06" rpy="0.0 0 0.0"/>
   </xacro:mid360>

File: LIO-SAM_MID360_ROS2_PKG/ros2/src/ros2_livox_simulation/urdf/my_robot/sensor/mid360.xacro (robot description, xacro)
@@ -24,5 +24,5 @@
         <origin xyz="0.025 -0.0265 -0.025" rpy="${pi/2} 0 ${pi}"/>
         <geometry>
-          <mesh filename="package://ros2_livox_simulation/meshes/mid360.stl" scale="0.0008 0.0008 0.0008"/>
+          <mesh filename="/home/ywj/dog_slam/LIO-SAM_MID360_ROS2_PKG/ros2/src/ros2_livox_simulation/meshes/mid360.stl" scale="0.0008 0.0008 0.0008"/>
         </geometry>
       </visual>
@@ -30,5 +30,5 @@
     <origin xyz="0.025 -0.0265 -0.025" rpy="${pi/2} 0 ${pi}"/>
     <geometry>
-      <mesh filename="package://ros2_livox_simulation/meshes/mid360.stl" scale="0.0008 0.0008 0.0008"/>
+      <mesh filename="/home/ywj/dog_slam/LIO-SAM_MID360_ROS2_PKG/ros2/src/ros2_livox_simulation/meshes/mid360.stl" scale="0.0008 0.0008 0.0008"/>
     </geometry>
   </collision>
@@ -46,4 +46,6 @@
         <update_rate>10</update_rate>
         <plugin name="${name}_plugin" filename="libros2_livox.so">
+        <topic>${topic}</topic>
+        <xfer_format>1</xfer_format>  <!-- 设置为1表示Livox私有格式 -->
         <enable_intensity>true</enable_intensity>
         <intensity_mean>100</intensity_mean>  <!-- 强度均值（0-255，根据需求调整） -->

Commit message: 修正车轮脱离问题

File: LIO-SAM_MID360_ROS2_PKG/ros2/src/ros2_livox_simulation/urdf/my_robot/my_robot.xacro (robot description, xacro)
@@ -18,5 +18,5 @@
 <!-- =============== 轮子配置 =============== -->
     <xacro:cylinder_xacro
-    name="bhind_left_wheel"
+    name="behind_left_wheel"
     length="0.032"
     radius="0.04"
@@ -29,5 +29,5 @@
     axis_xyz="0 1 0"/>
     <xacro:cylinder_xacro
-    name="bhind_right_wheel"
+    name="behind_right_wheel"
     length="0.032"
     radius="0.04"
@@ -94,3 +94,9 @@
 <xacro:my_robot_ros2_control_planar />   <!-- 如果gazebo_control更改名字，请修改此处 -->
 <xacro:gazebo_sensor_plugin />
+<!-- gazebo_ros2_control plugin -->
+<gazebo>
+  <plugin name="gazebo_ros2_control" filename="libgazebo_ros2_control.so">
+    <parameters>/home/ywj/dog_slam/LIO-SAM_MID360_ROS2_PKG/ros2/install/ros2_livox_simulation/share/ros2_livox_simulation/config/myrobot_ros2_controller.yaml</parameters>
+  </plugin>
+</gazebo>
 </robot>

File: LIO-SAM_MID360_ROS2_PKG/ros2/src/ros2_livox_simulation/urdf/my_robot/plugins/gazebo_control_plugin.xacro (robot description, xacro)
@@ -7,4 +7,37 @@
                 <plugin>gazebo_ros2_control/GazeboSystem</plugin>
             </hardware>
+            <!-- 定义关节接口 -->
+            <joint name="behind_left_wheel_joint">
+                <command_interface name="velocity">
+                    <param name="min">-1</param>
+                    <param name="max">1</param>
+                </command_interface>
+                <state_interface name="position"/>
+                <state_interface name="velocity"/>
+            </joint>
+            <joint name="behind_right_wheel_joint">
+                <command_interface name="velocity">
+                    <param name="min">-1</param>
+                    <param name="max">1</param>
+                </command_interface>
+                <state_interface name="position"/>
+                <state_interface name="velocity"/>
+            </joint>
+            <joint name="ahead_left_wheel_joint">
+                <command_interface name="velocity">
+                    <param name="min">-1</param>
+                    <param name="max">1</param>
+                </command_interface>
+                <state_interface name="position"/>
+                <state_interface name="velocity"/>
+            </joint>
+            <joint name="ahead_right_wheel_joint">
+                <command_interface name="velocity">
+                    <param name="min">-1</param>
+                    <param name="max">1</param>
+                </command_interface>
+                <state_interface name="position"/>
+                <state_interface name="velocity"/>
+            </joint>
         </ros2_control>
         <gazebo>

File: LIO-SAM_MID360_ROS2_PKG/ros2/src/ros2_livox_simulation/urdf/my_robot/sensor/mid360.xacro (robot description, xacro)
@@ -46,13 +46,13 @@
         <update_rate>10</update_rate>
         <plugin name="${name}_plugin" filename="libros2_livox.so">
-        <topic>${topic}</topic>
-        <xfer_format>1</xfer_format>  <!-- 设置为1表示Livox私有格式 -->
-        <enable_intensity>true</enable_intensity>
-        <intensity_mean>100</intensity_mean>  <!-- 强度均值（0-255，根据需求调整） -->
-      <intensity_stddev>5</intensity_stddev>  <!-- 强度噪声（模拟真实波动） -->
+          <topic>${topic}</topic>
+          <xfer_format>1</xfer_format>  <!-- 设置为1表示Livox私有格式 -->
+          <enable_intensity>true</enable_intensity>
+          <intensity_mean>100</intensity_mean>  <!-- 强度均值（0-255，根据需求调整） -->
+          <intensity_stddev>0</intensity_stddev>  <!-- 强度噪声（模拟真实波动） -->
           <ray>
             <scan>
               <horizontal>
-                <samples>100</samples>
+                <samples>10</samples>
                 <resolution>1</resolution>
                 <min_angle>${0}</min_angle>
@@ -60,5 +60,5 @@
               </horizontal>
               <vertical>
-                <samples>360</samples>
+                <samples>36</samples>
                 <resolution>1</resolution>
                 <min_angle>${-7.22/180*M_PI}</min_angle>
@@ -79,5 +79,5 @@
           <visualize>false</visualize>
           <samples>${samples}</samples>
-          <downsample>10</downsample>
+          <downsample>5</downsample>
           <csv_file_name>$(find ros2_livox_simulation)/scan_mode/mid360.csv</csv_file_name>
           <topic>${topic}</topic>
