Commit message: 优化自动导航相关

File: LIO-SAM_MID360_ROS2_PKG/ros2/src/livox_gazebo_ros2_gpu_simulation/urdf/my_robot/plugins/gazebo_control_plugin.xacro (robot description, xacro)
@@ -50,5 +50,5 @@
                 </ros>
                 <!-- 频率 -->
-                <update_rate>40</update_rate>
+                <update_rate>100</update_rate>
                 <!-- 里程计frame id -->
                 <odometry_frame>odom</odometry_frame>
@@ -57,5 +57,5 @@
                 <!-- 是否发布里程计tf -->
                 <publish_odom_tf>false</publish_odom_tf>
-                <robot_base_frame>base_footprint</robot_base_frame>
+                <robot_base_frame>base_link</robot_base_frame>
                 <!-- 最大速度 -->
                 <max_vel_x>5.0</max_vel_x>

File: LIO-SAM_MID360_ROS2_PKG/ros2/src/livox_gazebo_ros2_gpu_simulation/urdf/my_robot/sensor/mid360.xacro (robot description, xacro)
@@ -8,5 +8,5 @@
   <xacro:property name="noise_mean" value="0.0"/>
   <xacro:property name="noise_stddev" value="0.002"/>
-  <xacro:property name="imu_update_rate" value="40"/>
+  <xacro:property name="imu_update_rate" value="100"/>
   <xacro:property name="gyro_noise_stddev" value="2e-4"/>
   <xacro:property name="accel_noise_stddev" value="1.7e-2"/>
@@ -48,10 +48,10 @@
         <visualize>false</visualize>
         <update_rate>10</update_rate>
-        <use_strict_rate>false</use_strict_rate>
+        <use_strict_rate>true</use_strict_rate>
         <plugin name="${name}_plugin" filename="liblivox_sim_gpu_laser.so">
           <visualize>false</visualize>
           <frameName>${name}</frameName>
           <samples>${samples}</samples>
-          <downsample>10</downsample>
+          <downsample>1</downsample>
           <csv_file_name>package://livox_gazebo_ros2_gpu_simulation/scan_mode/mid360.csv</csv_file_name>
           <topic>${topic}</topic>
@@ -60,5 +60,5 @@
           <scan>
             <horizontal>
-              <samples>360</samples>
+              <samples>180</samples>
               <resolution>1</resolution>
               <min_angle>${0}</min_angle>
@@ -66,5 +66,5 @@
             </horizontal>
             <vertical>
-              <samples>59</samples>
+              <samples>30</samples>
               <resolution>1</resolution>
               <min_angle>${-7.22/180*M_PI}</min_angle>
@@ -85,5 +85,6 @@
       </sensor>
       <sensor name="${name}_imu" type="imu">
-        <pose>0 0 0 0 0 0</pose> <always_on>true</always_on>
+        <pose>0 0 0 0 0 0</pose>
+        <always_on>true</always_on>
         <update_rate>${imu_update_rate}</update_rate>
         <visualize>false</visualize>
