Commit message: 优化gazebo发布频率

File: LIO-SAM_MID360_ROS2_PKG/ros2/src/livox_gazebo_ros2_gpu_simulation/urdf/mid360.xacro (robot description, xacro)
@@ -40,5 +40,5 @@
         <pose>0 0 0 0 0 0</pose>
         <visualize>false</visualize>
-        <update_rate>100</update_rate>
+        <update_rate>10</update_rate>
         <use_strict_rate>true</use_strict_rate>
         <plugin name="${name}_plugin" filename="liblivox_sim_gpu_laser.so">
@@ -78,5 +78,6 @@
       </sensor>
       <sensor name="${name}_imu" type="imu">
-        <pose>0 0 0 0 0 0</pose> <always_on>true</always_on>
+        <pose>0 0 0 0 0 0</pose>
+        <!-- <always_on>true</always_on> -->
         <update_rate>${imu_update_rate}</update_rate>
         <visualize>false</visualize>

File: LIO-SAM_MID360_ROS2_PKG/ros2/src/livox_gazebo_ros2_gpu_simulation/urdf/my_robot/my_robot.xacro (robot description, xacro)
@@ -63,10 +63,10 @@
 <!-- =============== 轮子配置 =============== -->
 <!-- =============== mid360 ============ -->
-  <xacro:mid360  name="livox_frame" parent="base_link" topic="/livox/lidar">
+  <xacro:mid360  name="livox_frame" parent="base_link" topic="/livox/lidar" imu_topic="/livox/imu" >
     <origin xyz="0.07 0.0 0.10" rpy="0 0 0"/>
   </xacro:mid360>
 <!-- =============== mid360 ============ -->
   <!-- =============== 传感器 ============ -->
-    <xacro:box_xacro
+    <!-- <xacro:box_xacro
         name="imu_link"
         length="0.02"
@@ -76,5 +76,5 @@
         is_child="true"
         parent_link="base_link"
-        xyz="0 0 0.02" />
+        xyz="0 0 0.02" /> -->
     <!-- <xacro:box_xacro
         name="camera_link"

File: LIO-SAM_MID360_ROS2_PKG/ros2/src/livox_gazebo_ros2_gpu_simulation/urdf/my_robot/plugins/gazebo_sensor_plugin.xacro (robot description, xacro)
@@ -2,74 +2,7 @@
 <robot xmlns:xacro="http://www.ros.org/wiki/xacro">
     <xacro:macro name="gazebo_sensor_plugin">
-<gazebo reference="imu_link">
-    <sensor name="imu_sensor" type="imu">
-        <plugin name="imu_plugin" filename="libgazebo_ros_imu_sensor.so">
-            <ros>
-                <namespace>/</namespace>
-                <remapping>~/out:=/livox/imu</remapping>
-            </ros>
-            <initial_orientation_as_reference>false</initial_orientation_as_reference>
-        </plugin>
-        <update_rate>100</update_rate>
-        <always_on>true</always_on>
-        <!-- 六轴噪声设置 -->
-        <imu>
-            <angular_velocity>
-                <x>
-                    <noise type="gaussian">
-                        <mean>0.0</mean>
-                        <stddev>2e-4</stddev>
-                        <bias_mean>0.0000075</bias_mean>
-                        <bias_stddev>0.0000008</bias_stddev>
-                    </noise>
-                </x>
-                <y>
-                    <noise type="gaussian">
-                        <mean>0.0</mean>
-                        <stddev>2e-4</stddev>
-                        <bias_mean>0.0000075</bias_mean>
-                        <bias_stddev>0.0000008</bias_stddev>
-                    </noise>
-                </y>
-                <z>
-                    <noise type="gaussian">
-                        <mean>0.0</mean>
-                        <stddev>2e-4</stddev>
-                        <bias_mean>0.0000075</bias_mean>
-                        <bias_stddev>0.0000008</bias_stddev>
-                    </noise>
-                </z>
-            </angular_velocity>
-            <linear_acceleration>
-                <x>
-                    <noise type="gaussian">
-                        <mean>0.0</mean>
-                        <stddev>1.7e-2</stddev>
-                        <bias_mean>0.1</bias_mean>
-                        <bias_stddev>0.001</bias_stddev>
-                    </noise>
-                </x>
-                <y>
-                    <noise type="gaussian">
-                        <mean>0.0</mean>
-                        <stddev>1.7e-2</stddev>
-                        <bias_mean>0.1</bias_mean>
-                        <bias_stddev>0.001</bias_stddev>
-                    </noise>
-                </y>
-                <z>
-                    <noise type="gaussian">
-                        <mean>0.0</mean>
-                        <stddev>1.7e-2</stddev>
-                        <bias_mean>0.1</bias_mean>
-                        <bias_stddev>0.001</bias_stddev>
-                    </noise>
-                </z>
-            </linear_acceleration>
-        </imu>
-    </sensor>
-</gazebo>
+        <!-- 独立的IMU传感器已被移除，使用mid360激光雷达内置的IMU -->
     </xacro:macro>
-<gazebo reference="camera_link">
+<!-- <gazebo reference="camera_link">
     <sensor type="depth" name="camera_sensor">
         <plugin name="depth_camera" filename="libgazebo_ros_camera.so">
@@ -95,4 +28,4 @@
         </camera>
     </sensor>
-</gazebo>
+</gazebo> -->
 </robot>

File: LIO-SAM_MID360_ROS2_PKG/ros2/src/livox_gazebo_ros2_gpu_simulation/urdf/my_robot/sensor/mid360.xacro (robot description, xacro)
@@ -8,5 +8,4 @@
   <xacro:property name="noise_mean" value="0.0"/>
   <xacro:property name="noise_stddev" value="0.002"/>
-  <xacro:property name="imu_update_rate" value="200"/>
   <xacro:property name="gyro_noise_stddev" value="2e-40"/>
   <xacro:property name="accel_noise_stddev" value="1.7e-20"/>
@@ -22,5 +21,5 @@
     </inertial>
   </xacro:macro>
-  <xacro:macro name="mid360" params="name:='' parent:= 'base_link' topic:='mid360' imu_topic:='imu/data' *origin ">
+  <xacro:macro name="mid360" params="name:='' parent:= 'base_link' topic:='/livox/lidar' imu_topic:='/livox/imu' *origin ">
     <link name="${name}">
       <visual>
@@ -48,9 +47,9 @@
         <visualize>false</visualize>
         <update_rate>10</update_rate>
-        <use_strict_rate>false</use_strict_rate>
+        <use_strict_rate>true</use_strict_rate>
         <plugin name="${name}_plugin" filename="liblivox_sim_gpu_laser.so">
           <visualize>false</visualize>
           <frameName>${name}</frameName>
-          <samples>10000</samples>
+          <samples>${samples}</samples>
           <downsample>1</downsample>
           <csv_file_name>package://livox_gazebo_ros2_gpu_simulation/scan_mode/mid360.csv</csv_file_name>
@@ -60,5 +59,5 @@
           <scan>
             <horizontal>
-              <samples>360</samples>
+              <samples>180</samples>
               <resolution>1</resolution>
               <min_angle>${0}</min_angle>
@@ -66,5 +65,5 @@
             </horizontal>
             <vertical>
-              <samples>120</samples>
+              <samples>30</samples>
               <resolution>1</resolution>
               <min_angle>${-7.22/180*M_PI}</min_angle>
@@ -87,5 +86,6 @@
         <pose>0 0 0 0 0 0</pose>
         <always_on>true</always_on>
-        <update_rate>100</update_rate>
+        <update_rate>40</update_rate>
+        <use_strict_rate>true</use_strict_rate>
         <visualize>false</visualize>
         <plugin name="${name}_imu_plugin" filename="libgazebo_ros_imu_sensor.so">
@@ -93,5 +93,7 @@
             <namespace>/</namespace>
             <output_type>sensor_msgs/msg/Imu</output_type>
-            <topic_name>${imu_topic}</topic_name> <frame_id>${name}</frame_id>
+            <topic_name>${imu_topic}</topic_name>
+            <remapping>~/out:=/livox/imu</remapping>
+            <frame_id>${name}</frame_id>
           </ros>
           <imu>
