Commit message: sync

File: LIO-SAM_MID360_ROS2_PKG/ros2/src/livox_gazebo_ros2_gpu_simulation/urdf/my_robot/sensor/mid360.xacro (robot description, xacro)
@@ -8,5 +8,5 @@
   <xacro:property name="noise_mean" value="0.0"/>
   <xacro:property name="noise_stddev" value="0.002"/>
-  <xacro:property name="imu_update_rate" value="200"/>
+  <xacro:property name="imu_update_rate" value="40"/>
   <xacro:property name="gyro_noise_stddev" value="2e-4"/>
   <xacro:property name="accel_noise_stddev" value="1.7e-2"/>
@@ -48,10 +48,10 @@
         <visualize>false</visualize>
         <update_rate>10</update_rate>
-        <use_strict_rate>true</use_strict_rate>
+        <use_strict_rate>false</use_strict_rate>
         <plugin name="${name}_plugin" filename="liblivox_sim_gpu_laser.so">
           <visualize>false</visualize>
           <frameName>${name}</frameName>
           <samples>${samples}</samples>
-          <downsample>5</downsample>
+          <downsample>10</downsample>
           <csv_file_name>package://livox_gazebo_ros2_gpu_simulation/scan_mode/mid360.csv</csv_file_name>
           <topic>${topic}</topic>
@@ -60,5 +60,5 @@
           <scan>
             <horizontal>
-              <samples>3600</samples>
+              <samples>360</samples>
               <resolution>1</resolution>
               <min_angle>${0}</min_angle>

Commit message: sync

File: LIO-SAM_MID360_ROS2_PKG/ros2/src/livox_gazebo_ros2_gpu_simulation/urdf/my_robot/sensor/mid360.xacro (robot description, xacro)
@@ -5,5 +5,5 @@
   <xacro:property name="laser_max_range" value="100.0"/>
   <xacro:property name="samples" value="10000"/>
-  <xacro:property name="resolution" value="0.002"/>
+  <xacro:property name="resolution" value="0.005"/>
   <xacro:property name="noise_mean" value="0.0"/>
   <xacro:property name="noise_stddev" value="0.002"/>
@@ -48,10 +48,10 @@
         <visualize>false</visualize>
         <update_rate>10</update_rate>
-        <use_strict_rate>true</use_strict_rate>
+        <use_strict_rate>false</use_strict_rate>
         <plugin name="${name}_plugin" filename="liblivox_sim_gpu_laser.so">
           <visualize>false</visualize>
           <frameName>${name}</frameName>
-          <samples>${samples}</samples>
-          <downsample>1</downsample>
+          <samples>10000</samples>
+          <downsample>10</downsample>
           <csv_file_name>package://livox_gazebo_ros2_gpu_simulation/scan_mode/mid360.csv</csv_file_name>
           <topic>${topic}</topic>
@@ -60,5 +60,5 @@
           <scan>
             <horizontal>
-              <samples>180</samples>
+              <samples>360</samples>
               <resolution>1</resolution>
               <min_angle>${0}</min_angle>
@@ -66,5 +66,5 @@
             </horizontal>
             <vertical>
-              <samples>30</samples>
+              <samples>59</samples>
               <resolution>1</resolution>
               <min_angle>${-7.22/180*M_PI}</min_angle>
@@ -77,9 +77,9 @@
             <resolution>${resolution}</resolution>
           </range>
-          <noise>
+          <!-- <noise>
             <type>gaussian</type>
             <mean>${noise_mean}</mean>
             <stddev>${noise_stddev}</stddev>
-          </noise>
+          </noise> -->
         </ray>
       </sensor>

Commit message: 添加多种lio算法

File: LIO-SAM_MID360_ROS2_PKG/ros2/src/livox_gazebo_ros2_gpu_simulation/urdf/my_robot/sensor/mid360.xacro (robot description, xacro)
@@ -3,7 +3,7 @@
   <xacro:property name="M_PI" value="3.1415926"/>
   <xacro:property name="laser_min_range" value="0.1"/>
-  <xacro:property name="laser_max_range" value="100.0"/>
-  <xacro:property name="samples" value="10000"/>
-  <xacro:property name="resolution" value="0.005"/>
+  <xacro:property name="laser_max_range" value="200.0"/>
+  <xacro:property name="samples" value="30000"/>
+  <xacro:property name="resolution" value="0.002"/>
   <xacro:property name="noise_mean" value="0.0"/>
   <xacro:property name="noise_stddev" value="0.002"/>
@@ -16,24 +16,24 @@
   <xacro:macro name="box_inertia" params="m w h d">
     <inertial>
-      <origin xyz="0 0 0" rpy="${M_PI/2} 0 ${M_PI/2}"/>
+      <origin xyz="0 0 0" rpy="${pi/2} 0 ${pi/2}"/>
       <mass value="${m}"/>
       <inertia ixx="${(m/12) * (h*h + d*d)}" ixy="0.0" ixz="0.0" iyy="${(m/12) * (w*w + d*d)}" iyz="0.0" izz="${(m/12) * (w*w + h*h)}"/>
     </inertial>
   </xacro:macro>
-  <xacro:macro name="mid360" params="name:='' parent:= 'base_link' topic:='/livox/lidar' imu_topic:='/livox/imu' *origin ">
+  <xacro:macro name="mid360" params="name:='' parent:= 'base_link' topic:='mid360' imu_topic:='/livox/imu' *origin ">
     <link name="${name}">
       <visual>
-        <origin xyz="0 0 0" rpy="0 0 ${M_PI}"/>
+        <origin xyz="0.025 -0.0265 -0.025" rpy="${pi/2} 0 ${pi}"/>
         <geometry>
-          <mesh filename="file:///home/ywj/dog_slam/LIO-SAM_MID360_ROS2_PKG/ros2/src/livox_gazebo_ros2_gpu_simulation/meshes/mid-360-scaled.dae"/>
+          <mesh filename="package://ros2_livox_simulation/meshes/mid360.stl" scale="0.0008 0.0008 0.0008"/>
         </geometry>
       </visual>
-      <collision>
-        <origin xyz="0 0 0" rpy="0 0 ${M_PI}"/>
-        <geometry>
-          <mesh filename="file:///home/ywj/dog_slam/LIO-SAM_MID360_ROS2_PKG/ros2/src/livox_gazebo_ros2_gpu_simulation/meshes/mid-360-scaled.dae"/>
-        </geometry>
-      </collision>
-      <xacro:box_inertia m="${mass}" w="${width}" h="${height}" d="${length}"/>
+  <collision>
+    <origin xyz="0.025 -0.0265 -0.025" rpy="${pi/2} 0 ${pi}"/>
+    <geometry>
+      <mesh filename="package://ros2_livox_simulation/meshes/mid360.stl" scale="0.0008 0.0008 0.0008"/>
+    </geometry>
+  </collision>
+   <xacro:box_inertia m="${mass}" w="${width}" h="${height}" d="${length}"/>
     </link>
     <joint name="${name}_joint" type="fixed">
@@ -43,43 +43,46 @@
     </joint>
     <gazebo reference="${name}">
-      <sensor type="gpu_ray" name="${name}_lidar">
+      <sensor type="ray" name="${name}">
         <pose>0 0 0 0 0 0</pose>
-        <visualize>false</visualize>
+        <visualize>true</visualize>
         <update_rate>10</update_rate>
-        <use_strict_rate>true</use_strict_rate>
-        <plugin name="${name}_plugin" filename="liblivox_sim_gpu_laser.so">
+        <plugin name="${name}_plugin" filename="libros2_livox.so">
+          <topic>${topic}</topic>
+          <xfer_format>1</xfer_format>  <!-- 设置为1表示Livox私有格式 -->
+          <enable_intensity>true</enable_intensity>
+          <intensity_mean>100</intensity_mean>  <!-- 强度均值（0-255，根据需求调整） -->
+          <intensity_stddev>0</intensity_stddev>  <!-- 强度噪声（模拟真实波动） -->
+          <ray>
+            <scan>
+              <horizontal>
+                <samples>10</samples>
+                <resolution>1</resolution>
+                <min_angle>${0}</min_angle>
+                <max_angle>${2*M_PI}</max_angle>
+              </horizontal>
+              <vertical>
+                <samples>36</samples>
+                <resolution>1</resolution>
+                <min_angle>${-7.22/180*M_PI}</min_angle>
+                <max_angle>${55.22/180*M_PI}</max_angle>
+              </vertical>
+            </scan>
+            <range>
+              <min>${laser_min_range}</min>
+              <max>${laser_max_range}</max>
+              <resolution>${resolution}</resolution>
+            </range>
+            <noise>
+              <type>gaussian</type>
+              <mean>${noise_mean}</mean>
+              <stddev>${noise_stddev}</stddev>
+            </noise>
+          </ray>
           <visualize>false</visualize>
-          <frameName>${name}</frameName>
           <samples>${samples}</samples>
-          <downsample>1</downsample>
-          <csv_file_name>package://livox_gazebo_ros2_gpu_simulation/scan_mode/mid360.csv</csv_file_name>
+          <downsample>5</downsample>
+          <csv_file_name>$(find ros2_livox_simulation)/scan_mode/mid360.csv</csv_file_name>
           <topic>${topic}</topic>
         </plugin>
-        <ray>
-          <scan>
-            <horizontal>
-              <samples>180</samples>
-              <resolution>1</resolution>
-              <min_angle>${0}</min_angle>
-              <max_angle>${2*M_PI}</max_angle>
-            </horizontal>
-            <vertical>
-              <samples>30</samples>
-              <resolution>1</resolution>
-              <min_angle>${-7.22/180*M_PI}</min_angle>
-              <max_angle>${55.22/180*M_PI}</max_angle>
-            </vertical>
-          </scan>
-          <range>
-            <min>${laser_min_range}</min>
-            <max>${laser_max_range}</max>
-            <resolution>${resolution}</resolution>
-          </range>
-          <noise>
-            <type>gaussian</type>
-            <mean>${noise_mean}</mean>
-            <stddev>${noise_stddev}</stddev>
-          </noise>
-        </ray>
       </sensor>
       <sensor name="${name}_imu" type="imu">
@@ -110,6 +113,6 @@
           </imu>
         </plugin>
-        </sensor>
-      </gazebo>
+      </sensor>
+    </gazebo>
   </xacro:macro>
 </robot>
