Commit message: fix

File: LIO-SAM_MID360_ROS2_PKG/ros2/src/livox_gazebo_ros2_gpu_simulation/urdf/my_robot/sensor/mid360_gpu.xacro (robot description, xacro)
@@ -4,5 +4,5 @@
   <xacro:property name="laser_min_range" value="0.1"/>
   <xacro:property name="laser_max_range" value="100.0"/>
-  <xacro:property name="samples" value="10000"/>
+  <xacro:property name="samples" value="20000"/>
   <xacro:property name="resolution" value="0.005"/>
   <xacro:property name="noise_mean" value="0.0"/>
@@ -59,5 +59,5 @@
           <scan>
             <horizontal>
-              <samples>180</samples>
+              <samples>360</samples>
               <resolution>1</resolution>
               <min_angle>${0}</min_angle>
@@ -65,5 +65,5 @@
             </horizontal>
             <vertical>
-              <samples>30</samples>
+              <samples>60</samples>
               <resolution>1</resolution>
               <min_angle>${-7.22/180*M_PI}</min_angle>
