Commit message: 多种调整

File: LIO-SAM_MID360_ROS2_PKG/ros2/src/livox_gazebo_ros2_gpu_simulation/urdf/my_robot/my_robot.xacro (robot description, xacro)
@@ -77,5 +77,5 @@
         parent_link="base_link"
         xyz="0 0 0.02" />
-    <xacro:box_xacro
+    <!-- <xacro:box_xacro
         name="camera_link"
         length="0.02"
@@ -85,5 +85,5 @@
         is_child="true"
         parent_link="base_link"
-        xyz="0.1 0.0 0.05"/>
+        xyz="0.1 0.0 0.05"/> -->
   <!-- =============== 传感器 ============ -->
 <!-- =============== 导入gazebo插件 ============ -->

File: LIO-SAM_MID360_ROS2_PKG/ros2/src/livox_gazebo_ros2_gpu_simulation/urdf/my_robot/sensor/mid360.xacro (robot description, xacro)
@@ -8,7 +8,7 @@
   <xacro:property name="noise_mean" value="0.0"/>
   <xacro:property name="noise_stddev" value="0.002"/>
-  <xacro:property name="imu_update_rate" value="100"/>
-  <xacro:property name="gyro_noise_stddev" value="2e-4"/>
-  <xacro:property name="accel_noise_stddev" value="1.7e-2"/>
+  <xacro:property name="imu_update_rate" value="200"/>
+  <xacro:property name="gyro_noise_stddev" value="2e-40"/>
+  <xacro:property name="accel_noise_stddev" value="1.7e-20"/>
   <xacro:property name="mass" value="0.4" />
   <xacro:property name="length" value="0.1" />
@@ -47,5 +47,5 @@
         <pose>0 0 0 0 0 0</pose>
         <visualize>false</visualize>
-        <update_rate>10</update_rate>
+        <update_rate>99</update_rate>
         <use_strict_rate>false</use_strict_rate>
         <plugin name="${name}_plugin" filename="liblivox_sim_gpu_laser.so">
@@ -53,5 +53,5 @@
           <frameName>${name}</frameName>
           <samples>10000</samples>
-          <downsample>10</downsample>
+          <downsample>3</downsample>
           <csv_file_name>package://livox_gazebo_ros2_gpu_simulation/scan_mode/mid360.csv</csv_file_name>
           <topic>${topic}</topic>
@@ -77,9 +77,9 @@
             <resolution>${resolution}</resolution>
           </range>
-          <!-- <noise>
+          <noise>
             <type>gaussian</type>
             <mean>${noise_mean}</mean>
             <stddev>${noise_stddev}</stddev>
-          </noise> -->
+          </noise>
         </ray>
       </sensor>

Commit message: keep last 1

File: LIO-SAM_MID360_ROS2_PKG/ros2/src/livox_gazebo_ros2_gpu_simulation/urdf/my_robot/my_robot.xacro (robot description, xacro)
@@ -64,5 +64,5 @@
 <!-- =============== mid360 ============ -->
   <xacro:mid360  name="livox_frame" parent="base_link" topic="/livox/lidar" imu_topic="/livox/imu" >
-    <origin xyz="0.07 0.0 0.10" rpy="0 0 0"/>
+    <origin xyz="0.07 0.0 0.10" rpy="0 0.5235987756 0"/>
   </xacro:mid360>
 <!-- =============== mid360 ============ -->

File: LIO-SAM_MID360_ROS2_PKG/ros2/src/livox_gazebo_ros2_gpu_simulation/urdf/my_robot/sensor/mid360_cpu.xacro (robot description, xacro)
@@ -26,5 +26,5 @@
         <origin xyz="0.025 -0.0265 -0.025" rpy="${pi/2} 0 ${pi}"/>
         <geometry>
-          <mesh filename="package://ros2_livox_simulation/meshes/mid360.stl" scale="0.0008 0.0008 0.0008"/>
+          <mesh filename="package://livox_gazebo_ros2_gpu_simulation/meshes/mid360.stl" scale="0.0008 0.0008 0.0008"/>
         </geometry>
       </visual>
@@ -32,5 +32,5 @@
     <origin xyz="0.025 -0.0265 -0.025" rpy="${pi/2} 0 ${pi}"/>
     <geometry>
-      <mesh filename="package://ros2_livox_simulation/meshes/mid360.stl" scale="0.0008 0.0008 0.0008"/>
+      <mesh filename="package://livox_gazebo_ros2_gpu_simulation/meshes/mid360.stl" scale="0.0008 0.0008 0.0008"/>
     </geometry>
   </collision>
@@ -82,5 +82,5 @@
           <samples>${samples}</samples>
           <downsample>5</downsample>
-          <csv_file_name>$(find ros2_livox_simulation)/scan_mode/mid360.csv</csv_file_name>
+          <csv_file_name>$(find livox_gazebo_ros2_gpu_simulation)/scan_mode/mid360.csv</csv_file_name>
           <topic>${topic}</topic>
         </plugin>
@@ -89,5 +89,5 @@
         <pose>0 0 0 0 0 0</pose>
         <always_on>true</always_on>
-        <update_rate>40</update_rate>
+        <update_rate>200</update_rate>
         <use_strict_rate>true</use_strict_rate>
         <visualize>false</visualize>
