Commit message: gazebo7可正常运行，删除旧gazebo版本

File: LIO-SAM_MID360_ROS2_PKG/ros2/src/livox_gazebo_garden/urdf/my_robot/my_robot.urdf (robot description, URDF)
Before this commit: robot mid360_robot, 7 links, 6 joints
Joints:
- joint livox_frame_joint: origin xyz=0.07 0.0 0.10 rpy=0 0.5235987756 0 -> xyz=0.07 0.0 0.10 rpy=0 0 0

File: LIO-SAM_MID360_ROS2_PKG/ros2/src/livox_gazebo_garden/urdf/my_robot/my_robot.xacro (robot description, xacro)
@@ -26,5 +26,5 @@
     is_child="true"
     parent_link="base_link"
-    xyz="-0.08 0.07 -0.04"
+    xyz="-0.12 0.07 -0.04"
     axis_xyz="0 1 0"/>
     <xacro:cylinder_xacro
@@ -37,5 +37,5 @@
     is_child="true"
     parent_link="base_link"
-    xyz="-0.08 -0.07 -0.04"
+    xyz="-0.12 -0.07 -0.04"
     axis_xyz="0 1 0"/>
     <xacro:cylinder_xacro
@@ -48,5 +48,5 @@
     is_child="true"
     parent_link="base_link"
-    xyz="0.08 0.07 -0.04"
+    xyz="0.12 0.07 -0.04"
     axis_xyz="0 1 0"/>
     <xacro:cylinder_xacro
@@ -59,5 +59,5 @@
     is_child="true"
     parent_link="base_link"
-    xyz="0.08 -0.07 -0.04"
+    xyz="0.12 -0.07 -0.04"
     axis_xyz="0 1 0"/>
 <!-- =============== 轮子配置 =============== -->

File: LIO-SAM_MID360_ROS2_PKG/ros2/src/livox_gazebo_garden/urdf/my_robot/plugins/gazebo_control_plugin.xacro (robot description, xacro)
@@ -6,4 +6,6 @@
                 <left_joint>behind_left_wheel_joint</left_joint>
                 <right_joint>behind_right_wheel_joint</right_joint>
+                <left_joint>ahead_left_wheel_joint</left_joint>
+                <right_joint>ahead_right_wheel_joint</right_joint>
                 <wheel_separation>0.14</wheel_separation>
                 <wheel_radius>0.04</wheel_radius>

Commit message: 同步修改

File: LIO-SAM_MID360_ROS2_PKG/ros2/src/livox_gazebo_garden/urdf/my_robot/my_robot.urdf (robot description, URDF)
Before this commit: robot mid360_robot, 7 links, 6 joints
Joints:
- joint livox_frame_joint: origin xyz=0.07 0.0 0.10 rpy=0 0 0 -> xyz=0.07 0.0 0.10 rpy=0 0.5236 0

File: LIO-SAM_MID360_ROS2_PKG/ros2/src/livox_gazebo_garden/urdf/my_robot/my_robot.xacro (robot description, xacro)
@@ -64,5 +64,5 @@
 <!-- =============== mid360 ============ -->
   <xacro:mid360  name="livox_frame" parent="base_link" topic="/livox/lidar" imu_topic="/livox/imu" >
-    <origin xyz="0.07 0.0 0.10" rpy="0 0.5235987756 0"/>
+    <origin xyz="0.07 0.0 0.10" rpy="0 0.5236 0"/>
   </xacro:mid360>
 <!-- =============== mid360 ============ -->
